Commit message: turn dae from Z_UP to Y_UP

File: resources/robots/go2/urdf/arx5go2.urdf (robot description, URDF)
Before this commit: robot go2_description, 39 links, 38 joints
Links:
- removed link imu
- removed link radar
Joints:
- removed joint imu_joint
- removed joint radar_joint

Commit message: fixed arxgo2 urdf

File: resources/robots/go2/urdf/arx5go2.urdf (robot description, URDF)
Before this commit: robot go2_description, 37 links, 36 joints
Joints:
- joint FL_calf_joint: limit lower=-2.7227 upper=-0.83776 effort=45.43 velocity=15.70 -> lower=-2.7227 upper=-0.83776 effort=23.7 velocity=15.70
- joint FR_calf_joint: limit lower=-2.7227 upper=-0.83776 effort=45.43 velocity=15.70 -> lower=-2.7227 upper=-0.83776 effort=23.7 velocity=15.70
- joint RL_calf_joint: limit lower=-2.7227 upper=-0.83776 effort=45.43 velocity=15.70 -> lower=-2.7227 upper=-0.83776 effort=23.7 velocity=15.70
- joint RR_calf_joint: limit lower=-2.7227 upper=-0.83776 effort=45.43 velocity=15.70 -> lower=-2.7227 upper=-0.83776 effort=23.7 velocity=15.70
